File: electronics/araneo-mainboard/araneo-mainboard.kicad_sch (KiCad schematic)
At the start: 58 parts, among them J1 GPIO, J2 OLED, SW1 SW, U1 IMU, U2 L78M05CDT, U3 BD9C601EFJ, U4 POWER, U5 PAM8403D

Commit message: electronics: add footprints
Parts:
- C15, C16, C18: footprint (none) -> Capacitor_SMD:C_0603_1608Metric_Pad1.08x0.95mm_HandSolder
- C17: footprint (none) -> Capacitor_THT:CP_Radial_D10.0mm_P5.00mm
- C2: footprint Capacitor_SMD:C_0603_1608Metric_Pad1.08x0.95mm_HandSolder -> Capacitor_SMD:C_0805_2012Metric_Pad1.18x1.45mm_HandSolder
- FB1, FB2: footprint (none) -> Resistor_SMD:R_0603_1608Metric_Pad0.98x0.95mm_HandSolder
- LS1: footprint Connector_Molex:Molex_PicoBlade_53398-0271_1x02-1MP_P1.25mm_Vertical -> PCM_SparkFun-Connector:ScrewTerminal_1x02_P3.5mm_Blue
- R2: value 7.8k -> 7.87k
Connections:
- net +3V3: no longer C9.1
- net GND: now also C9.1
Other:
- moved on the sheet: C9
Changed lines of the file:
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@@
 	)
 	(junction
-		(at 153.67 76.2)
-		(diameter 0)
-		(color 0 0 0 0)
-	)
-	(junction
 		(at 213.36 102.87)
 		(diameter 0)
@@
 	)
 	(junction
+		(at 163.83 76.2)
+		(diameter 0)
+		(color 0 0 0 0)
+	)
+	(junction
 		(at 133.35 45.72)
 		(diameter 0)
@@
 		(color 0 0 0 0)
 	)
-	(junction
-		(at 161.29 76.2)
-		(diameter 0)
-		(color 0 0 0 0)
-	)
 	(no_connect
 		(at 113.03 149.86)
@@
 	(wire
 		(pts
+			(xy 163.83 76.2) (xy 161.29 76.2)
+		)
+		(stroke
+			(width 0)
+			(type default)
+		)
+	)
+	(wire
+		(pts
 			(xy 105.41 151.13) (xy 100.33 151.13)
 		)
@@
 	(wire
 		(pts
-			(xy 161.29 76.2) (xy 161.29 85.09)
-		)
-		(stroke
-			(width 0)
-			(type default)
-		)
-	)
-	(wire
-		(pts
 			(xy 158.75 134.62) (xy 167.64 134.62)
 		)
@@
 	(wire
 		(pts
-			(xy 153.67 85.09) (xy 153.67 76.2)
-		)
-		(stroke
-			(width 0)
-			(type default)
-		)
-	)
-	(wire
-		(pts
 			(xy 200.66 114.3) (xy 200.66 113.03)
 		)
@@
 	(wire
 		(pts
-			(xy 171.45 76.2) (xy 161.29 76.2)
+			(xy 171.45 76.2) (xy 163.83 76.2)
 		)
 		(stroke
@@
 		)
 	)
+	(wire
+		(pts
+			(xy 163.83 83.82) (xy 163.83 85.09)
+		)
+		(stroke
+			(width 0)
+			(type default)
+		)
+	)
 	(image
 		(at 86.36 19.05)
@@
 			)
 		)
-		(property "Footprint" ""
+		(property "Footprint" "Resistor_SMD:R_0603_1608Metric_Pad0.98x0.95mm_HandSolder"
 			(at 229.87 123.698 90)
 			(hide yes)
@@
 			)
 		)
-		(property "Value" "7.8k"
+		(property "Value" "7.87k"
 			(at 80.01 69.85 0)
 			(show_name no)
@@
 			)
 		)
-		(property "Footprint" ""
+		(property "Footprint" "Capacitor_SMD:C_0603_1608Metric_Pad1.08x0.95mm_HandSolder"
 			(at 207.3148 102.87 0)
 			(hide yes)
@@
 	)
 	(symbol
+		(lib_id "power:GND")
+		(at 163.83 85.09 0)
+		(unit 1)
+		(body_style 1)
+		(exclude_from_sim no)
+		(in_bom yes)
+		(on_board yes)
+		(in_pos_files yes)
+		(dnp no)
+		(fields_autoplaced yes)
+		(property "Reference" "#PWR037"
+			(at 163.83 91.44 0)
+			(hide yes)
+			(show_name no)
+			(do_not_autoplace no)
+			(effects
+				(font
+					(size 1.27 1.27)
+				)
+			)
+		)
+		(property "Value" "GND"
+			(at 163.83 90.17 0)
+			(show_name no)
+			(do_not_autoplace no)
+			(effects
+				(font
+					(size 1.27 1.27)
+				)
+			)
+		)
+		(property "Footprint" ""
+			(at 163.83 85.09 0)
+			(hide yes)
+			(show_name no)
+			(do_not_autoplace no)
+			(effects
+				(font
+					(size 1.27 1.27)
+				)
+			)
+		)
+		(property "Datasheet" ""
+			(at 163.83 85.09 0)
+			(hide yes)
+			(show_name no)
+			(do_not_autoplace no)
+			(effects
+				(font
+					(size 1.27 1.27)
+				)
+			)
+		)
+		(property "Description" "Power symbol creates a global label with name \"GND\" , ground"
+			(at 163.83 85.09 0)
+			(hide yes)
+			(show_name no)
+			(do_not_autoplace no)
+			(effects
+				(font
+					(size 1.27 1.27)
+				)
+			)
+		)
+		(pin "1"
+		)
+		(instances
+			(project "araneo-mainboard"
+				(path "/0ff7269e-d15c-4d73-8399-8898e55a410d"
+					(reference "#PWR037")
+					(unit 1)
+				)
+			)
+		)
+	)
+	(symbol
 		(lib_id "Amplifier_Audio:PAM8403D")
 		(at 210.82 129.54 0)
@@
 			)
 		)
-		(property "Footprint" ""
+		(property "Footprint" "Capacitor_SMD:C_0603_1608Metric_Pad1.08x0.95mm_HandSolder"
 			(at 221.2848 102.87 0)
 			(hide yes)
@@
 			)
 		)
-		(property "Footprint" ""
+		(property "Footprint" "Capacitor_THT:CP_Radial_D10.0mm_P5.00mm"
 			(at 212.3948 102.87 0)
 			(hide yes)
@@
 			)
 		)
-		(property "Footprint" "Capacitor_SMD:C_0603_1608Metric_Pad1.08x0.95mm_HandSolder"
+		(property "Footprint" "Capacitor_SMD:C_0805_2012Metric_Pad1.18x1.45mm_HandSolder"
 			(at 165.1 61.2648 0)
 			(hide yes)
@@
 			)
 		)
-		(property "Footprint" ""
+		(property "Footprint" "Resistor_SMD:R_0603_1608Metric_Pad0.98x0.95mm_HandSolder"
 			(at 236.22 126.238 90)
 			(hide yes)
@@
 			)
 		)
-		(property "Footprint" ""
+		(property "Footprint" "Capacitor_SMD:C_0603_1608Metric_Pad1.08x0.95mm_HandSolder"
 			(at 199.6948 105.41 0)
 			(hide yes)
@@
 	(symbol
 		(lib_id "Device:C")
-		(at 157.48 85.09 90)
+		(at 163.83 80.01 180)
 		(unit 1)
 		(body_style 1)
@@
 		(dnp no)
 		(property "Reference" "C9"
-			(at 157.48 81.28 90)
+			(at 160.528 82.296 0)
 			(show_name no)
 			(do_not_autoplace no)
@@
 		)
 		(property "Value" "100nF"
-			(at 158.242 89.154 90)
+			(at 168.148 83.058 0)
 			(show_name no)
 			(do_not_autoplace no)
@@
 		)
 		(property "Footprint" "Capacitor_SMD:C_0603_1608Metric_Pad1.08x0.95mm_HandSolder"
-			(at 161.29 84.1248 0)
+			(at 162.8648 76.2 0)
 			(hide yes)
 			(show_name no)
@@
 		)
 		(property "Datasheet" ""
-			(at 157.48 85.09 0)
+			(at 163.83 80.01 0)
 			(hide yes)
 			(show_name no)
@@
 		)
 		(property "Description" "Unpolarized capacitor"
-			(at 157.48 85.09 0)
+			(at 163.83 80.01 0)
 			(hide yes)
 			(show_name no)
@@
 			)
 		)
-		(property "Footprint" "Connector_Molex:Molex_PicoBlade_53398-0271_1x02-1MP_P1.25mm_Vertical"
+		(property "Footprint" "PCM_SparkFun-Connector:ScrewTerminal_1x02_P3.5mm_Blue"
 			(at 259.08 127 0)
 			(hide yes)

Commit message: electronics: pcb v2
Connections:
- net +7.4V: no longer C2.1, C3.2, C4.2, D2.2 (A), SW1.1 (A), U2.1 (IN), U3.2 (VIN), U4.1 (Pin_1)
- net D1: now also A1.17 (GPIO13); no longer A1.11 (GPIO8)
- net D2: now also A1.19 (GPIO14); no longer A1.12 (GPIO9)
- net D3: now also A1.20 (GPIO15); no longer A1.14 (GPIO10)
- net GPIO12: now also J1.4 (Pin_4); no longer J1.1 (Pin_1)
- net GPIO22: now also J1.7 (Pin_7); no longer J1.5 (Pin_5)
- net SCL_IMU: now also A1.32 (GPIO27_ADC1); no longer A1.22 (GPIO17)
- net SDA_IMU: now also A1.31 (GPIO26_ADC0); no longer A1.21 (GPIO16)
- net GPIO13 renamed GPIO9
- net GPIO9: now also A1.12 (GPIO9); no longer A1.17 (GPIO13)
- net GPIO14 renamed GPIO10
- net GPIO10: now also A1.14 (GPIO10); no longer A1.19 (GPIO14)
- removed net GPIO15: A1.20 (GPIO15), J1.4 (Pin_4)
- net GPIO26 renamed GPIO17
- net GPIO17: now also A1.22 (GPIO17); no longer A1.31 (GPIO26_ADC0)
- removed net GPIO27: A1.32 (GPIO27_ADC1), J1.7 (Pin_7)
- new net +7.4V_F: C2.1, C3.2, C4.2, D2.2 (A), SW1.1 (A), U2.1 (IN), U3.2 (VIN), U4.1 (Pin_1)
- new net GPIO16: A1.21 (GPIO16), J1.5 (Pin_5)
- new net GPIO8: A1.11 (GPIO8), J1.1 (Pin_1)

Commit message: electronics: board pcb
Parts:
- removed J1: GPIO, Connector_PinHeader_2.54mm:PinHeader_1x08_P2.54mm_Vertical, symbol Connector:Conn_01x08_Pin
- removed LED1: Diode1, Connector_PinHeader_2.54mm:PinHeader_1x02_P2.54mm_Vertical, symbol Connector:Conn_01x02_Pin
- removed LED2: Diode2, Connector_PinHeader_2.54mm:PinHeader_1x02_P2.54mm_Vertical, symbol Connector:Conn_01x02_Pin
- removed LED3: Diode3, Connector_PinHeader_2.54mm:PinHeader_1x02_P2.54mm_Vertical, symbol Connector:Conn_01x02_Pin
- removed R4, R5, R6: 4.7k, Resistor_SMD:R_0603_1608Metric_Pad0.98x0.95mm_HandSolder, symbol Device:R
- added D3: DEBUG_LED, PCM_SparkFun-LED:LED_0603_1608Metric, symbol PCM_SparkFun-LED:LED
- added H5: MountingHole, MountingHole:MountingHole_2.1mm, symbol Mechanical:MountingHole
- added J1: GPIO, Connector_PinHeader_2.54mm:PinHeader_1x09_P2.54mm_Vertical, symbol Connector:Conn_01x09_Pin
- added R10: 4.7k, Resistor_SMD:R_0603_1608Metric_Pad0.98x0.95mm_HandSolder, symbol Device:R
- added R11: 10k, Resistor_SMD:R_0603_1608Metric_Pad0.98x0.95mm_HandSolder, symbol Device:R
- added R13: 1k, Resistor_SMD:R_0603_1608Metric_Pad0.98x0.95mm_HandSolder, symbol Device:R
- D2: value POWER_LED -> BUCK_LED
- J2: footprint Connector_PinHeader_2.54mm:PinHeader_1x04_P2.54mm_Vertical -> PCM_SparkFun-Connector:ScrewTerminal_1x04_P3.5mm_Locking
- SW1: footprint Connector_PinHeader_2.54mm:PinHeader_1x02_P2.54mm_Vertical -> PCM_SparkFun-Connector:ScrewTerminal_1x02_P5.0mm
Connections:
- net +3V3: now also J2.4 (Pin_4); no longer J2.1 (Pin_1)
- net +7.4V: now also F1.1, U4.1 (Pin_1); no longer F1.2
- net +7.4V_F: now also SW1.2 (B), R11.1; no longer SW1.1 (A), U4.1 (Pin_1)
- net D1: now also D3.2 (A)
- net GND: now also J2.3 (Pin_3), R10.2, R13.2; no longer J2.2 (Pin_2)
- net GPIO10: now also J1.3 (Pin_3)
- net GPIO12: now also J1.4 (Pin_4)
- net GPIO16: now also J1.7 (Pin_7)
- net GPIO17: now also J1.8 (Pin_8)
- net GPIO22: now also J1.9 (Pin_9)
- net GPIO8: now also J1.1 (Pin_1)
- net GPIO9: now also J1.2 (Pin_2)
- net SCL_OLED: now also J2.2 (Pin_2); no longer J2.3 (Pin_3)
- net SDA_OLED: now also J2.1 (Pin_1); no longer J2.4 (Pin_4)
- net D2 renamed GPIO14
- net GPIO14: now also J1.5 (Pin_5)
- net D3 renamed GPIO15
- net GPIO15: now also J1.6 (Pin_6)
- net GPIO28 renamed MEASURE
- net MEASURE: now also R10.1, R11.2
- new net: F1.2, SW1.1 (A)
- new net: D3.1 (K), R13.1
Other:
- note added: "TO do - uzupełnić zakupy (rezystory, terminatory, led) - przycisk oled"
