File: electronics/araneo-mainboard/imu.kicad_sch (KiCad schematic)
At the start: 7 parts, among them IC2 BMI270

Commit message: electronics: add 100n capacitors
Changed lines of the file:
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@@
-		(color 0 0 0 0)
-	)
-	(junction
-		(at 90.17 48.26)
-		(diameter 0)
 		(color 0 0 0 0)
 	)
@@
 	(wire
 		(pts
-			(xy 83.82 54.61) (xy 87.63 54.61)
-		)
-		(stroke
-			(width 0)
-			(type default)
-		)
-	)
-	(wire
-		(pts
-			(xy 90.17 50.8) (xy 90.17 48.26)
-		)
-		(stroke
-			(width 0)
-			(type default)
-		)
-	)
-	(wire
-		(pts
 			(xy 93.98 48.26) (xy 101.6 48.26)
 		)
@@
 	(wire
 		(pts
-			(xy 87.63 54.61) (xy 87.63 50.8)
-		)
-		(stroke
-			(width 0)
-			(type default)
-		)
-	)
-	(wire
-		(pts
 			(xy 101.6 48.26) (xy 104.14 48.26)
 		)
@@
 	(wire
 		(pts
-			(xy 62.23 76.2) (xy 83.82 76.2)
+			(xy 62.23 73.66) (xy 71.12 73.66)
 		)
 		(stroke
@@
 	(wire
 		(pts
-			(xy 62.23 76.2) (xy 62.23 73.66)
-		)
-		(stroke
-			(width 0)
-			(type default)
-		)
-	)
-	(wire
-		(pts
 			(xy 66.04 66.04) (xy 66.04 67.31)
 		)
@@
 	(wire
 		(pts
-			(xy 87.63 50.8) (xy 90.17 50.8)
-		)
-		(stroke
-			(width 0)
-			(type default)
-		)
-	)
-	(wire
-		(pts
 			(xy 64.77 21.59) (xy 64.77 22.86)
 		)
@@
 	(wire
 		(pts
-			(xy 90.17 48.26) (xy 93.98 48.26)
-		)
-		(stroke
-			(width 0)
-			(type default)
-		)
-	)
-	(wire
-		(pts
 			(xy 93.98 60.96) (xy 93.98 57.15)
 		)
@@
 	(wire
 		(pts
-			(xy 88.9 48.26) (xy 90.17 48.26)
+			(xy 88.9 48.26) (xy 93.98 48.26)
 		)
 		(stroke
@@
 		(pts
 			(xy 101.6 55.88) (xy 101.6 57.15)
-		)
-		(stroke
-			(width 0)
-			(type default)
-		)
-	)
-	(wire
-		(pts
-			(xy 83.82 76.2) (xy 83.82 54.61)
 		)
 		(stroke
@@
 					(unit 1)
 				)
+			)
+		)
+	)
+	(symbol
+		(lib_id "power:+3.3V")
+		(at 71.12 73.66 0)
+		(unit 1)
+		(body_style 1)
+		(exclude_from_sim no)
+		(in_bom yes)
+		(on_board yes)
+		(in_pos_files yes)
+		(dnp no)
+		(property "Reference" "#PWR089"
+			(at 71.12 77.47 0)
+			(hide yes)
+			(show_name no)
+			(do_not_autoplace no)
+			(effects
+				(font
+					(size 1.27 1.27)
+				)
+			)
+		)
+		(property "Value" "+3V3"
+			(at 75.184 69.596 0)
+			(show_name no)
+			(do_not_autoplace no)
+			(effects
+				(font
+					(size 1.27 1.27)
+				)
+			)
+		)
+		(property "Footprint" ""
+			(at 71.12 73.66 0)
+			(hide yes)
+			(show_name no)
+			(do_not_autoplace no)
+			(effects
+				(font
+					(size 1.27 1.27)
+				)
+			)
+		)
+		(property "Datasheet" ""
+			(at 71.12 73.66 0)
+			(hide yes)
+			(show_name no)
+			(do_not_autoplace no)
+			(effects
+				(font
+					(size 1.27 1.27)
+				)
+			)
+		)
+		(property "Description" "Power symbol creates a global label with name \"+3.3V\""
+			(at 71.12 73.66 0)
+			(hide yes)
+			(show_name no)
+			(do_not_autoplace no)
+			(effects
+				(font
+					(size 1.27 1.27)
+				)
+			)
+		)
+		(pin "1"
+		)
+		(instances
+			(project "araneo-mainboard"
+				(path "/0ff7269e-d15c-4d73-8399-8898e55a410d/0c8726fa-3d9d-4f6c-bd2a-acab0879e92f"
+					(reference "#PWR089")
+					(unit 1)
+				)

Commit message: electronics: remove unnecessary capacitors, add net labels, change screw terminal to JST_XH
Connections:
- net +3V3: no longer C42.2, C43.2
- net VDD_IMU: now reaches FB4.1, IC2.8 (VDD)
- net VDD_IMU: now also C42.2, C43.2
Other:
- moved on the sheet: FB4
